Commit message: addednew config files

File: urdf/sensors_setup.urdf (robot description, URDF)
Before this commit: robot sensors_setup, 5 links, 4 joints
Links:
- removed link imu
- added link imu_link
Joints:
- joint base_link_to_imu: child imu -> imu_link
- joint imu_to_camera: parent imu -> imu_link
